File: pcb/tinyI2C.brd (EAGLE design)
At the start: 83.2 x 83.2 mm, 29 parts, among them IC1 IC_TTL_74_125, IC2 TPS73618(0.4A), U1 LPC824M201JHI33, X1 TSW-112-02-S-S, X2 TSW-106-02-S-S-RA, X3 TSW-112-02-S-S, X4 TSW-102-02-S-S, X5 TSW-102-02-S-S

Commit message: [ PCB ] trace change and panelize
Parts:
- moved R6 0.50 mm to (3.60, 22.3)
- moved R7 0.50 mm to (3.60, 19.7)
- moved R8 0.50 mm to (3.60, 17.1)
- moved R9 0.50 mm to (3.60, 14.6)
Routing:
- net 1.8V: track 53.9 -> 54.7 mm

Commit message: [ PCB ][ BRD ] new header for ISP
added ISP header next to RESET header
removed trace to X1[3]
moved R3 to near th header
silkn name and bottom VDD trace change
Parts:
- added X6: TSW-102-02-S-S, con-samtec.local:TSW-102-02-S-S
- X2: value TSW-106-02-S-S-RA -> TSW-112-02-S-S; device con-samtec.local:TSW-106-02-S-S-RA -> con-samtec.local:TSW-112-02-S-S
- X3: value TSW-112-02-S-S -> TSW-106-02-S-S-RA; device con-samtec.local:TSW-112-02-S-S -> con-samtec.local:TSW-106-02-S-S-RA
- moved R3 21.3 mm to (10.3, 13.6), turned to 180 degrees
- moved X2 15.7 mm to (19.0, 26.0), turned to 90 degrees
- moved X3 15.7 mm to (10.1, 39.0), turned to 180 degrees
- moved R1 0.54 mm to (3.60, 29.4), turned to 180 degrees
- moved R10 0.50 mm to (3.60, 13.0)
- moved R2 0.41 mm to (3.60, 25.7)
Connections:
- net !ISP!: now also X6.1; no longer X1.3
- net 5V: now also X3.3; no longer X2.3
- net CTS<-: now also X3.2; no longer X2.2
- net GND: now also X3.1, X6.2; no longer X2.1
- net GPIO00: now also X2.1; no longer X3.1
- net GPIO01: now also X2.2; no longer X3.2
- net GPIO02: now also X2.3; no longer X3.3
- net GPIO03: now also X2.4; no longer X3.4
- net GPIO04: now also X2.5; no longer X3.5
- net GPIO05: now also X2.6; no longer X3.6
- net GPIO06: now also X2.7; no longer X3.7
- net GPIO07: now also X2.8; no longer X3.8
- net RTS->: now also X3.6; no longer X2.6
- net RX<-: now also X3.5; no longer X2.5
- net SPI_CS: now also X2.12; no longer X3.12
- net SPI_MISO: now also X2.10; no longer X3.10
- net SPI_MOSI: now also X2.9; no longer X3.9
- net SPI_SCK: now also X2.11; no longer X3.11
- net TX->: now also X3.4; no longer X2.4
Routing:
- net !ISP!: track 16.6 -> 25.1 mm
- net 1.8V: track 54.7 -> 50.0 mm, vias 14 -> 15
- net SPI_CS: track 19.6 -> 20.4 mm
- net GND: track 16.2 -> 15.4 mm
- net TGT_CTS: track 25.0 -> 24.3 mm

Commit message: [ PCB ][ BRD ] LDO and buffer replace
LDO replaced to MIC5355(Micron, 2 outputs, Vout1=3.3V, Vout2=1.8V) IC2
-> IC3
3.3V line added as LDO changed
3-state buffer replaced from 1x quad to 2x single
disconnect CTS, RTS
Parts:
- added C7: 1005, rcl:C1005
- added IC3: IC_LDO_MIC5355, mylib:IC_08_0.65_160MIL
- added TP6: TPTP07R, testpad:TP07R
- IC1: value IC_TTL_74_125 -> 74LVC1G125DCK; device mylib:DHVQFN14 -> 74xx-little-us:SC70-5
- IC2: value TPS73618(0.4A) -> 74LVC1G125DCK; device mylib:SOT95P280X145-5N -> 74xx-little-us:SC70-5
- moved IC2 9.20 mm to (15.5, 34.0), turned to 90 degrees
- moved TP1 5.92 mm to (3.00, 34.7)
- moved C3 5.17 mm to (9.10, 34.9)
- moved IC1 3.35 mm to (12.3, 34.6), turned to 90 degrees
- moved C1 3.00 mm to (13.8, 32.2), turned to 180 degrees
- moved C5 1.84 mm to (7.50, 35.6)
- moved TP3 1.53 mm to (5.10, 30.9)
- moved C4 1.08 mm to (7.10, 30.8)
- moved TP2 0.86 mm to (9.00, 33.0)
- moved R4 0.78 mm to (13.0, 28.5)
Connections:
- removed net CTS<-: IC1.6, X3.2
- removed net N$1: C3.1, IC2.4
- removed net RTS->: IC1.9, X3.6
- removed net TGT_CTS: IC1.8, U1.16
- removed net TGT_RTS: IC1.5, U1.1
- new net 3.3V: C3.1, C7.1, IC1.5, IC3.8, TP6.TP
- net 1.8V: now also IC3.7; no longer IC1.14
- net 5V: now also IC3.1, IC3.4, IC3.5; no longer IC2.1, IC2.3
- net GND: now also C7.2, IC1.3, IC2.1, IC2.3, IC3.2, IC3.EXP; no longer IC1.10, IC1.13, IC1.4, IC1.7, IC1.EXP, IC2.2
- net RX<-: now also IC1.4; no longer IC1.11
- net TGT_RX: now also IC2.4; no longer IC1.3
- net TGT_TX: now also IC1.2; no longer IC1.12
- net TX->: now also IC2.2; no longer IC1.2
Routing:
- net TGT_CTS: track 24.3 -> 0.00 mm, vias 2 -> 0
- net CTS<-: track 14.0 -> 0.00 mm
- net TGT_RTS: track 10.8 -> 0.00 mm, vias 2 -> 0
- net RTS->: track 8.70 -> 0.00 mm
- net GND: track 15.4 -> 7.61 mm
- net TGT_TX: track 16.1 -> 9.95 mm, vias 2 -> 0
- net TX->: track 5.50 -> 10.4 mm
- net RX<-: track 8.40 -> 3.67 mm, vias 0 -> 1
- net 1.8V: track 50.0 -> 46.5 mm, vias 15 -> 14
- net 3.3V: track 0.00 -> 2.13 mm
- net 5V: track 8.12 -> 10.00 mm
- net N$1: track 1.71 -> 0.00 mm
- net !RESET!: track 17.8 -> 16.2 mm
- net TGT_RX: track 18.5 -> 17.8 mm
- added copper zone on layer 1, net 1.8V
- added copper zone on layer 1, net 3.3V
- added copper zone on layer 1, net 5V

Commit message: [ PCB ][ SCH ] new header X7 X7[1] = P0_13 X7[2] = P0_1
Parts:
- added X7: TSW-102-02-S-S, con-samtec.local:TSW-102-02-S-S
- IC1, IC2: device 74xx-little-us:SC70-5 -> 74xx-little-us_local:SC70-5
- moved R3 14.0 mm to (12.8, 27.4), turned to 0 degrees
- moved X6 4.02 mm to (13.9, 17.1), turned to 90 degrees
- moved R4 0.63 mm to (12.8, 29.1)
Connections:
- new net P0_1: U1.16, X7.2
- new net P0_13: U1.1, X7.1
Routing:
- net P0_13: track 0.00 -> 20.3 mm, vias 0 -> 1
- net P0_1: track 0.00 -> 18.8 mm
- net !ISP!: track 25.1 -> 15.8 mm, vias 2 -> 1
- net TGT_RX: track 17.8 -> 21.0 mm
- net !RESET!: track 16.2 -> 19.2 mm, vias 2 -> 1
- net 1.8V: track 46.5 -> 45.0 mm
- net SPI_CS: track 20.4 -> 19.5 mm
- net SPI_MISO: track 9.92 -> 10.7 mm
- net GPIO03: track 12.5 -> 11.9 mm
- net GPIO02: track 14.5 -> 14.0 mm
- net GPIO00: track 18.2 -> 17.7 mm
- net GND: vias 13 -> 14
Other:
- board text added: "!ISP"
- board text added: "!RST"

Commit message: [ PCB ][ BRD ] R and C library replace
standard rcl to mylib
Parts:
- C1, C2, C3, C4, C6, C7: device rcl:C1005 -> mylib:C0402
- C5: value 1608 -> 1005; device rcl:C0402 -> mylib:C0402
- R1, R10, R2, R3, R4, R5, R6, R7, R8, R9: device rcl:R1005 -> mylib:C0402
Changed lines of the file:
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@@
 <attribute name="VALUE" x="5.8" y="25.9" size="1.27" layer="27" ratio="10" rot="R270"/>
 </element>
-<element name="C1" library="rcl" package="C1005" value="1005" x="13.8" y="32.2" smashed="yes" rot="R180">
+<element name="C1" library="mylib" package="C0402" value="1005" x="13.8" y="32.2" smashed="yes" rot="R180">
 <attribute name="NAME" x="13.965" y="30.535" size="1" layer="25" font="vector" ratio="15"/>
 <attribute name="VALUE" x="14.435" y="34.105" size="1.27" layer="27" rot="R180"/>
 </element>
-<element name="C2" library="rcl" package="C1005" value="1005" x="9.7" y="17.9" smashed="yes" rot="R270">
+<element name="C2" library="mylib" package="C0402" value="1005" x="9.7" y="17.9" smashed="yes" rot="R270">
 <attribute name="NAME" x="9.065" y="16.165" size="1.27" layer="25" font="vector" ratio="15" rot="R90"/>
 <attribute name="VALUE" x="7.795" y="18.535" size="1.27" layer="27" rot="R270"/>
 </element>
-<element name="C4" library="rcl" package="C1005" value="1005" x="7.1" y="30.8" smashed="yes" rot="R180">
+<element name="C4" library="mylib" package="C0402" value="1005" x="7.1" y="30.8" smashed="yes" rot="R180">
 <attribute name="NAME" x="9.465" y="29.935" size="1" layer="25" font="vector" ratio="15"/>
 <attribute name="VALUE" x="7.735" y="32.705" size="1.27" layer="27" rot="R180"/>
 </element>
-<element name="C5" library="rcl" package="C0402" value="1608" x="7.5" y="35.6" smashed="yes" rot="R270">
+<element name="C5" library="mylib" package="C0402" value="1005" x="7.5" y="35.6" smashed="yes" rot="R270">
 <attribute name="NAME" x="6.765" y="34.765" size="1" layer="25" font="vector" ratio="15" rot="R90"/>
 <attribute name="VALUE" x="5.595" y="36.235" size="1.27" layer="27" rot="R270"/>
@@
 <attribute name="VALUE" x="4.846" y="30.392" size="0.0254" layer="27"/>
 </element>
-<element name="R1" library="rcl" package="R1005" value="220/1005" x="3.6" y="29.4" smashed="yes" rot="R180">
+<element name="R1" library="mylib" package="C0402" value="220/1005" x="3.6" y="29.4" smashed="yes" rot="R180">
 <attribute name="NAME" x="2.565" y="30.035" size="1.2" layer="25" font="vector" ratio="15"/>
 <attribute name="VALUE" x="4.235" y="31.305" size="1.27" layer="27" rot="R180"/>
 </element>
-<element name="R2" library="rcl" package="R1005" value="220/1005" x="3.6" y="25.7" smashed="yes" rot="R180">
+<element name="R2" library="mylib" package="C0402" value="220/1005" x="3.6" y="25.7" smashed="yes" rot="R180">
 <attribute name="NAME" x="4.865" y="25.335" size="1.2" layer="25" font="vector" ratio="15"/>
 <attribute name="VALUE" x="4.235" y="27.605" size="1.27" layer="27" rot="R180"/>
 </element>
-<element name="R3" library="rcl" package="R1005" value="10k/1005" x="12.8" y="27.4" smashed="yes">
+<element name="R3" library="mylib" package="C0402" value="10k/1005" x="12.8" y="27.4" smashed="yes">
 <attribute name="NAME" x="13.965" y="26.035" size="1.016" layer="25" font="vector" ratio="15"/>
 <attribute name="VALUE" x="12.165" y="25.495" size="1.27" layer="27"/>
 </element>
-<element name="R4" library="rcl" package="R1005" value="10k/1005" x="12.8" y="29.1" smashed="yes">
+<element name="R4" library="mylib" package="C0402" value="10k/1005" x="12.8" y="29.1" smashed="yes">
 <attribute name="NAME" x="11.865" y="29.735" size="1" layer="25" font="vector" ratio="15"/>
 <attribute name="VALUE" x="12.165" y="27.195" size="1.27" layer="27"/>
 </element>
-<element name="R5" library="rcl" package="R1005" value="10k/1005" x="3.6" y="24.4" smashed="yes" rot="R180">
+<element name="R5" library="mylib" package="C0402" value="10k/1005" x="3.6" y="24.4" smashed="yes" rot="R180">
 <attribute name="NAME" x="4.865" y="23.735" size="1.2" layer="25" font="vector" ratio="15"/>
 <attribute name="VALUE" x="4.235" y="26.305" size="1.27" layer="27" rot="R180"/>
 </element>
-<element name="R6" library="rcl" package="R1005" value="10k/1005" x="3.6" y="22.3" smashed="yes" rot="R180">
+<element name="R6" library="mylib" package="C0402" value="10k/1005" x="3.6" y="22.3" smashed="yes" rot="R180">
 <attribute name="NAME" x="4.865" y="21.735" size="1.2" layer="25" font="vector" ratio="15"/>
 <attribute name="VALUE" x="4.235" y="24.205" size="1.27" layer="27" rot="R180"/>
 </element>
-<element name="R7" library="rcl" package="R1005" value="10k/1005" x="3.6" y="19.7" smashed="yes" rot="R180">
+<element name="R7" library="mylib" package="C0402" value="10k/1005" x="3.6" y="19.7" smashed="yes" rot="R180">
 <attribute name="NAME" x="5.165" y="19.135" size="1.2" layer="25" font="vector" ratio="15"/>
 <attribute name="VALUE" x="4.235" y="21.605" size="1.27" layer="27" rot="R180"/>
 </element>
-<element name="R8" library="rcl" package="R1005" value="10k/1005" x="3.6" y="17.1" smashed="yes" rot="R180">
+<element name="R8" library="mylib" package="C0402" value="10k/1005" x="3.6" y="17.1" smashed="yes" rot="R180">
 <attribute name="NAME" x="5.165" y="16.535" size="1.2" layer="25" font="vector" ratio="15"/>
 <attribute name="VALUE" x="4.235" y="19.005" size="1.27" layer="27" rot="R180"/>
 </element>
-<element name="R9" library="rcl" package="R1005" value="10k/1005" x="3.6" y="14.6" smashed="yes" rot="R180">
+<element name="R9" library="mylib" package="C0402" value="10k/1005" x="3.6" y="14.6" smashed="yes" rot="R180">
 <attribute name="NAME" x="5.165" y="14.335" size="1.2" layer="25" font="vector" ratio="15"/>
 <attribute name="VALUE" x="4.235" y="16.505" size="1.27" layer="27" rot="R180"/>
 </element>
-<element name="R10" library="rcl" package="R1005" value="10k/1005" x="3.6" y="13" smashed="yes" rot="R180">
+<element name="R10" library="mylib" package="C0402" value="10k/1005" x="3.6" y="13" smashed="yes" rot="R180">
 <attribute name="NAME" x="5.165" y="12.835" size="1.2" layer="25" font="vector" ratio="15"/>
 <attribute name="VALUE" x="4.235" y="14.905" size="1.27" layer="27" rot="R180"/>
 </element>
-<element name="C3" library="rcl" package="C1005" value="1005" x="9.1" y="34.9" smashed="yes" rot="R90">
+<element name="C3" library="mylib" package="C0402" value="1005" x="9.1" y="34.9" smashed="yes" rot="R90">
 <attribute name="NAME" x="10.365" y="31.065" size="1" layer="25" font="vector" ratio="15" rot="R90"/>
 <attribute name="VALUE" x="11.005" y="34.265" size="1.27" layer="27" rot="R90"/>
@@
 <attribute name="VALUE" x="20.26" y="43.145" size="1.27" layer="27" rot="R180"/>
 </element>
-<element name="C6" library="rcl" package="C1005" value="1005" x="11.3" y="17.9" smashed="yes" rot="R270">
+<element name="C6" library="mylib" package="C0402" value="1005" x="11.3" y="17.9" smashed="yes" rot="R270">
 <attribute name="NAME" x="10.265" y="14.835" size="1.2" layer="25" font="vector" ratio="15"/>
 <attribute name="VALUE" x="9.395" y="18.535" size="1.27" layer="27" rot="R270"/>
@@
 <attribute name="VALUE" x="18.04" y="31.46" size="1.27" layer="27" rot="R90"/>
 </element>
-<element name="C7" library="rcl" package="C1005" value="1005" x="10.3" y="34.9" smashed="yes" rot="R90">
+<element name="C7" library="mylib" package="C0402" value="1005" x="10.3" y="34.9" smashed="yes" rot="R90">
 <attribute name="NAME" x="11.465" y="31.065" size="1" layer="25" font="vector" ratio="15" rot="R90"/>
 <attribute name="VALUE" x="12.205" y="34.265" size="1.27" layer="27" rot="R90"/>
